File: led/leds65k_1.kicad_sch (KiCad schematic)
At the start: 32 parts, among them Q13 IPS70R1K4P7SAKMA1, Q2 IPS70R1K4P7SAKMA1, U1 LM397, U2 4N25, U5 4N25

Commit message: fixup
Parts:
- LED1, LED10, LED11, LED12, LED13, LED14, LED2, LED3, LED4, LED5, LED6, LED7, LED8, LED9: value L150-18705024000H0 -> L150-65705024000H0

Commit message: using single and dual top switch current driver circuits
Parts:
- removed D6, D7, D8, D9: 1N5408, Diode_THT:D_DO-41_SOD81_P10.16mm_Horizontal, symbol Diode:1N4007
- removed ESMR401VSN102MA50S_3: ESMR401VSN102MA50S, arduino-library:CAPPRD1000W180D3550H5250, symbol Device:C_Polarized
- removed Q13, Q2: IPS70R1K4P7SAKMA1, arduino-library:TO229P240X654X875-3P, symbol IPS70R1K4P7SAKMA1:IPS70R1K4P7SAKMA1
- removed R1: RSF1JT1R00, arduino-library:RESAD2900W85L1100D450, symbol RSF1JT1R00:RSF1JT1R00
- removed R4, R5, R6: MFR-25FTE52-100K, Resistor_THT:R_Axial_DIN0204_L3.6mm_D1.6mm_P2.54mm_Vertical, symbol Device:R
- removed RH2: MFR50SFTE52-1K, Resistor_THT:R_Axial_DIN0204_L3.6mm_D1.6mm_P2.54mm_Vertical, symbol Device:R
- removed TH1: CL60, Resistor_THT:R_Axial_DIN0516_L15.5mm_D5.0mm_P7.62mm_Vertical, symbol Device:Thermistor_NTC
- removed U1: LM397, Package_TO_SOT_SMD:SOT-23-5, symbol Comparator:LM397
- removed U2, U5: 4N25, Package_DIP:DIP-6_W7.62mm, symbol Isolator:4N25
- D1: renamed from D5; value 1.5KE440A -> zener; Mouser Part Number (none) -> 603-1.5KE440A/B
- L1: value HCTI-220-5.8 -> 220 uH @5.8A; Mouser Part Number (none) -> 530-HCTI-220-5.8
- renumbered LED5 to LED1, LED4 to LED2, LED2 to LED4, LED1 to LED5
Connections:
- net VDC-: now reaches L1.1, LED7.3 (K_2)
- net VDC+: now reaches D1.1 (K), LED8.4 (A_2)
Other:
- moved on the sheet: D1, L1, LED10, LED11, LED12, LED13, LED14, LED2, LED3, LED4, LED5, LED6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

Commit message: led pcb designed
Parts:
- added H2, H7: MountingHole_Pad, Connector_Pin:Pin_D1.0mm_L10.0mm_LooseFit, symbol Mechanical:MountingHole_Pad
- D1: footprint Diode_THT:D_DO-15_P5.08mm_Vertical_KathodeUp -> arduino-library:DIOM7959X262N; Mouser Part Number 603-1.5KE440A/B -> 833-SMCJ1.5KE440A-TP
- L1: footprint arduino-library:HCTI22058 -> arduino-library:Coil_6cmx1cm
Connections:
- net VDC+: now also H2.1
- net VDC-: now also H7.1
Changed lines of the file:
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@@
 	(paper "A4")
+	(junction
+		(at 71.12 45.72)
+		(diameter 0)
+		(color 0 0 0 0)
+	)
 	(junction
 		(at 97.79 21.59)
@@
 		(color 0 0 0 0)
 	)
+	(junction
+		(at 71.12 43.18)
+		(diameter 0)
+		(color 0 0 0 0)
+	)
 	(wire
 		(pts
@@
 	(wire
 		(pts
-			(xy 64.77 45.72) (xy 83.82 45.72)
+			(xy 64.77 45.72) (xy 71.12 45.72)
+		)
+		(stroke
+			(width 0)
+			(type default)
+		)
+	)
+	(wire
+		(pts
+			(xy 71.12 45.72) (xy 83.82 45.72)
 		)
 		(stroke
@@
 	(wire
 		(pts
+			(xy 71.12 43.18) (xy 82.55 43.18)
+		)
+		(stroke
+			(width 0)
+			(type default)
+		)
+	)
+	(wire
+		(pts
 			(xy 152.4 38.1) (xy 152.4 52.07)
 		)
@@
 	(wire
 		(pts
-			(xy 64.77 43.18) (xy 82.55 43.18)
+			(xy 64.77 43.18) (xy 71.12 43.18)
 		)
 		(stroke
@@
 	)
 	(symbol
+		(lib_id "Mechanical:MountingHole_Pad")
+		(at 71.12 48.26 180)
+		(unit 1)
+		(exclude_from_sim no)
+		(in_bom no)
+		(on_board yes)
+		(dnp no)
+		(fields_autoplaced yes)
+		(property "Reference" "H7"
+			(at 73.66 48.2599 0)
+			(effects
+				(font
+					(size 1.27 1.27)
+				)
+				(justify right)
+			)
+		)
+		(property "Value" "MountingHole_Pad"
+			(at 73.66 50.7999 0)
+			(effects
+				(font
+					(size 1.27 1.27)
+				)
+				(justify right)
+			)
+		)
+		(property "Footprint" "Connector_Pin:Pin_D1.0mm_L10.0mm_LooseFit"
+			(at 71.12 48.26 0)
+			(effects
+				(font
+					(size 1.27 1.27)
+				)
+				(hide yes)
+			)
+		)
+		(property "Datasheet" "~"
+			(at 71.12 48.26 0)
+			(effects
+				(font
+					(size 1.27 1.27)
+				)
+				(hide yes)
+			)
+		)
+		(property "Description" "Mounting Hole with connection"
+			(at 71.12 48.26 0)
+			(effects
+				(font
+					(size 1.27 1.27)
+				)
+				(hide yes)
+			)
+		)
+		(pin "1"
+		)
+		(instances
+			(project "led"
+				(path "/3f432d6c-3758-4345-b186-9310705dc61b/26342586-4ff5-45da-bd07-da6b77ca317c"
+					(reference "H11")
+					(unit 1)
+				)
+				(path "/3f432d6c-3758-4345-b186-9310705dc61b/6c4c63f0-577c-4e78-b127-3e8364c63f27"
+					(reference "H8")
+					(unit 1)
+				)
+				(path "/3f432d6c-3758-4345-b186-9310705dc61b/7a0af58d-8343-4daf-8db7-90bf6f6b226e"
+					(reference "H9")
+					(unit 1)
+				)
+				(path "/3f432d6c-3758-4345-b186-9310705dc61b/90c382e1-500b-4dd2-a1bc-dcf0e666755f"
+					(reference "H10")
+					(unit 1)
+				)
+				(path "/3f432d6c-3758-4345-b186-9310705dc61b/d9a700bb-2ef5-49e4-a53c-a5b54e2b049e"
+					(reference "H7")
+					(unit 1)
+				)
+			)
+		)
+	)
+	(symbol
 		(lib_id "Device:L")
 		(at 97.79 80.01 180)
@@
 			)
 		)
-		(property "Footprint" "arduino-library:HCTI22058"
+		(property "Footprint" "arduino-library:Coil_6cmx1cm"
 			(at 97.79 80.01 0)
 			(effects
@@
 			)
 		)
-		(property "Description" "Inductor"
+		(property "Description" "Inductor coil radius=1cm, length=5.5cm, turns=3*55=165, wire radius=1mm air or wood core"
 			(at 97.79 80.01 0)
 			(effects
@@
 	)
 	(symbol
+		(lib_id "Mechanical:MountingHole_Pad")
+		(at 71.12 40.64 0)
+		(unit 1)
+		(exclude_from_sim no)
+		(in_bom no)
+		(on_board yes)
+		(dnp no)
+		(fields_autoplaced yes)
+		(property "Reference" "H2"
+			(at 73.66 38.0999 0)
+			(effects
+				(font
+					(size 1.27 1.27)
+				)
+				(justify left)
+			)
+		)
+		(property "Value" "MountingHole_Pad"
+			(at 73.66 40.6399 0)
+			(effects
+				(font
+					(size 1.27 1.27)
+				)
+				(justify left)
+			)
+		)
+		(property "Footprint" "Connector_Pin:Pin_D1.0mm_L10.0mm_LooseFit"
+			(at 71.12 40.64 0)
+			(effects
+				(font
+					(size 1.27 1.27)
+				)
+				(hide yes)
+			)
+		)
+		(property "Datasheet" "~"
+			(at 71.12 40.64 0)
+			(effects
+				(font
+					(size 1.27 1.27)
+				)
+				(hide yes)
+			)
+		)
+		(property "Description" "Mounting Hole with connection"
+			(at 71.12 40.64 0)
+			(effects
+				(font
+					(size 1.27 1.27)
+				)
+				(hide yes)
+			)
+		)
+		(pin "1"
+		)
+		(instances
+			(project ""
+				(path "/3f432d6c-3758-4345-b186-9310705dc61b/26342586-4ff5-45da-bd07-da6b77ca317c"
+					(reference "H6")
+					(unit 1)
+				)
+				(path "/3f432d6c-3758-4345-b186-9310705dc61b/6c4c63f0-577c-4e78-b127-3e8364c63f27"
+					(reference "H3")
+					(unit 1)
+				)
+				(path "/3f432d6c-3758-4345-b186-9310705dc61b/7a0af58d-8343-4daf-8db7-90bf6f6b226e"
+					(reference "H4")
+					(unit 1)
+				)
+				(path "/3f432d6c-3758-4345-b186-9310705dc61b/90c382e1-500b-4dd2-a1bc-dcf0e666755f"
+					(reference "H5")
+					(unit 1)
+				)
+				(path "/3f432d6c-3758-4345-b186-9310705dc61b/d9a700bb-2ef5-49e4-a53c-a5b54e2b049e"
+					(reference "H2")
+					(unit 1)
+				)
+			)
+		)
+	)
+	(symbol
 		(lib_id "Device:D_Zener")
 		(at 97.79 72.39 270)
@@
 			)
 		)
-		(property "Footprint" "Diode_THT:D_DO-15_P5.08mm_Vertical_KathodeUp"
+		(property "Footprint" "arduino-library:DIOM7959X262N"
 			(at 97.79 72.39 0)
 			(effects
@@
 			)
 		)
-		(property "Datasheet" "https://www.littelfuse.com/assetdocs/tvs-diodes-1-5ke-datasheet?assetguid=9D02C7D2-86A5-4BFF-9251-966D6AF02BF7"
+		(property "Datasheet" "https://hu.mouser.com/datasheet/3/225/1/SMCJ1.5KE6.8(C)A-SMCJ1.5KE550(C)A(DO-214AB).pdf"
 			(at 97.79 72.39 0)
 			(effects
@@
 			)
 		)
-		(property "Mouser Part Number" "603-1.5KE440A/B"
+		(property "Mouser Part Number" "833-SMCJ1.5KE440A-TP"
 			(at 97.79 72.39 90)
 			(effects
