File: controller/RJ11.kicad_sch (KiCad schematic)
At the start: 10 parts, among them J15 6P6C, J16 6P6C, J17 6P6C, J18 6P6C, J19 6P6C, J20 6P6C, Q14 BS170, Q15 BS170

Commit message: sensors
Connections:
- net 1Wire: now also J15.6, J16.6, J17.6, J18.6, J19.6, J20.6; no longer J15.1, J16.1, J17.1, J18.1, J19.1, J20.1
- net 3V3: now also J15.2, J16.2, J17.2, J18.2, J19.2, J20.2; no longer J15.5, J16.5, J17.5, J18.5, J19.5, J20.5
- net 5V: now also J15.5, J16.5, J17.5, J18.5, J19.5, J20.5; no longer J15.2, J16.2, J17.2, J18.2, J19.2, J20.2
- net GND: now also J15.1, J16.1, J19.1, J20.1; no longer J15.6, J16.6, J19.6, J20.6
- net SCL: now also J15.4, J16.4, J17.4, J18.4, J19.4, J20.4; no longer J15.3, J16.3, J17.3, J18.3, J19.3, J20.3
- net SDA: now also J15.3, J16.3, J17.3, J18.3, J19.3, J20.3; no longer J15.4, J16.4, J17.4, J18.4, J19.4, J20.4
- net at Q15.1 (D): now also J18.1; no longer J18.6
- net at Q14.1 (D): now also J17.1; no longer J17.6
Other:
- moved on the sheet: J15, J16, J17, J18, J19, J20
Changed lines of the file:
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@@
 	(symbol
 		(lib_id "Connector:6P6C")
-		(at 95.25 152.4 90)
-		(unit 1)
-		(exclude_from_sim no)
-		(in_bom yes)
-		(on_board yes)
-		(dnp no)
-		(fields_autoplaced yes)
+		(at 92.71 152.4 270)
+		(mirror x)
+		(unit 1)
+		(exclude_from_sim no)
+		(in_bom yes)
+		(on_board yes)
+		(dnp no)
 		(property "Reference" "J16"
-			(at 104.14 151.1299 90)
+			(at 83.82 151.1299 90)
 			(effects
 				(font
@@
 		)
 		(property "Value" "6P6C"
-			(at 104.14 153.6699 90)
-			(effects
-				(font
-					(size 1.27 1.27)
-				)
-				(justify right)
-			)
-		)
-		(property "Footprint" ""
-			(at 94.615 152.4 90)
-			(effects
-				(font
-					(size 1.27 1.27)
-				)
-				(hide yes)
-			)
-		)
-		(property "Datasheet" "~"
-			(at 94.615 152.4 90)
+			(at 83.82 153.6699 90)
+			(effects
+				(font
+					(size 1.27 1.27)
+				)
+				(justify right)
+			)
+		)
+		(property "Footprint" ""
+			(at 93.345 152.4 90)
+			(effects
+				(font
+					(size 1.27 1.27)
+				)
+				(hide yes)
+			)
+		)
+		(property "Datasheet" "~"
+			(at 93.345 152.4 90)
 			(effects
 				(font
@@
 		)
 		(property "Description" "RJ connector, 6P6C (6 positions 6 connected), RJ12/RJ18/RJ25"
-			(at 95.25 152.4 0)
+			(at 92.71 152.4 0)
 			(effects
 				(font
@@
 	(symbol
 		(lib_id "Connector:6P6C")
-		(at 128.27 152.4 90)
-		(unit 1)
-		(exclude_from_sim no)
-		(in_bom yes)
-		(on_board yes)
-		(dnp no)
-		(fields_autoplaced yes)
+		(at 125.73 152.4 270)
+		(mirror x)
+		(unit 1)
+		(exclude_from_sim no)
+		(in_bom yes)
+		(on_board yes)
+		(dnp no)
 		(property "Reference" "J17"
-			(at 137.16 151.1299 90)
+			(at 116.84 151.1299 90)
 			(effects
 				(font
@@
 		)
 		(property "Value" "6P6C"
-			(at 137.16 153.6699 90)
-			(effects
-				(font
-					(size 1.27 1.27)
-				)
-				(justify right)
-			)
-		)
-		(property "Footprint" ""
-			(at 127.635 152.4 90)
-			(effects
-				(font
-					(size 1.27 1.27)
-				)
-				(hide yes)
-			)
-		)
-		(property "Datasheet" "~"
-			(at 127.635 152.4 90)
+			(at 116.84 153.6699 90)
+			(effects
+				(font
+					(size 1.27 1.27)
+				)
+				(justify right)
+			)
+		)
+		(property "Footprint" ""
+			(at 126.365 152.4 90)
+			(effects
+				(font
+					(size 1.27 1.27)
+				)
+				(hide yes)
+			)
+		)
+		(property "Datasheet" "~"
+			(at 126.365 152.4 90)
 			(effects
 				(font
@@
 		)
 		(property "Description" "RJ connector, 6P6C (6 positions 6 connected), RJ12/RJ18/RJ25"
-			(at 128.27 152.4 0)
+			(at 125.73 152.4 0)
 			(effects
 				(font
@@
 	(symbol
 		(lib_id "Connector:6P6C")
-		(at 62.23 151.13 90)
-		(unit 1)
-		(exclude_from_sim no)
-		(in_bom yes)
-		(on_board yes)
-		(dnp no)
-		(fields_autoplaced yes)
+		(at 59.69 151.13 270)
+		(mirror x)
+		(unit 1)
+		(exclude_from_sim no)
+		(in_bom yes)
+		(on_board yes)
+		(dnp no)
 		(property "Reference" "J15"
-			(at 71.12 149.8599 90)
+			(at 50.8 149.8599 90)
 			(effects
 				(font
@@
 		)
 		(property "Value" "6P6C"
-			(at 71.12 152.3999 90)
-			(effects
-				(font
-					(size 1.27 1.27)
-				)
-				(justify right)
-			)
-		)
-		(property "Footprint" ""
-			(at 61.595 151.13 90)
-			(effects
-				(font
-					(size 1.27 1.27)
-				)
-				(hide yes)
-			)
-		)
-		(property "Datasheet" "~"
-			(at 61.595 151.13 90)
+			(at 50.8 152.3999 90)
+			(effects
+				(font
+					(size 1.27 1.27)
+				)
+				(justify right)
+			)
+		)
+		(property "Footprint" ""
+			(at 60.325 151.13 90)
+			(effects
+				(font
+					(size 1.27 1.27)
+				)
+				(hide yes)
+			)
+		)
+		(property "Datasheet" "~"
+			(at 60.325 151.13 90)
 			(effects
 				(font
@@
 		)
 		(property "Description" "RJ connector, 6P6C (6 positions 6 connected), RJ12/RJ18/RJ25"
-			(at 62.23 151.13 0)
+			(at 59.69 151.13 0)
 			(effects
 				(font
@@
 	(symbol
 		(lib_id "Connector:6P6C")
-		(at 194.31 152.4 90)
-		(unit 1)
-		(exclude_from_sim no)
-		(in_bom yes)
-		(on_board yes)
-		(dnp no)
-		(fields_autoplaced yes)
+		(at 191.77 152.4 270)
+		(mirror x)
+		(unit 1)
+		(exclude_from_sim no)
+		(in_bom yes)
+		(on_board yes)
+		(dnp no)
 		(property "Reference" "J19"
-			(at 203.2 151.1299 90)
+			(at 182.88 151.1299 90)
 			(effects
 				(font
@@
 		)
 		(property "Value" "6P6C"
-			(at 203.2 153.6699 90)
-			(effects
-				(font
-					(size 1.27 1.27)
-				)
-				(justify right)
-			)
-		)
-		(property "Footprint" ""
-			(at 193.675 152.4 90)
-			(effects
-				(font
-					(size 1.27 1.27)
-				)
-				(hide yes)
-			)
-		)
-		(property "Datasheet" "~"
-			(at 193.675 152.4 90)
+			(at 182.88 153.6699 90)
+			(effects
+				(font
+					(size 1.27 1.27)
+				)
+				(justify right)
+			)
+		)
+		(property "Footprint" ""
+			(at 192.405 152.4 90)
+			(effects
+				(font
+					(size 1.27 1.27)
+				)
+				(hide yes)
+			)
+		)
+		(property "Datasheet" "~"
+			(at 192.405 152.4 90)
 			(effects
 				(font
@@
 		)
 		(property "Description" "RJ connector, 6P6C (6 positions 6 connected), RJ12/RJ18/RJ25"
-			(at 194.31 152.4 0)
+			(at 191.77 152.4 0)
 			(effects
 				(font
@@
 	(symbol
 		(lib_id "Connector:6P6C")
-		(at 161.29 152.4 90)
-		(unit 1)
-		(exclude_from_sim no)
-		(in_bom yes)
-		(on_board yes)
-		(dnp no)
-		(fields_autoplaced yes)
+		(at 158.75 152.4 270)
+		(mirror x)
+		(unit 1)
+		(exclude_from_sim no)
+		(in_bom yes)
+		(on_board yes)
+		(dnp no)
 		(property "Reference" "J18"
-			(at 170.18 151.1299 90)
+			(at 149.86 151.1299 90)
 			(effects
 				(font
@@
 		)
 		(property "Value" "6P6C"
-			(at 170.18 153.6699 90)
-			(effects
-				(font
-					(size 1.27 1.27)
-				)
-				(justify right)
-			)
-		)
-		(property "Footprint" ""
-			(at 160.655 152.4 90)
-			(effects
-				(font
-					(size 1.27 1.27)
-				)
-				(hide yes)
-			)
-		)
-		(property "Datasheet" "~"
-			(at 160.655 152.4 90)
+			(at 149.86 153.6699 90)
+			(effects
+				(font
+					(size 1.27 1.27)
+				)
+				(justify right)
+			)
+		)
+		(property "Footprint" ""
+			(at 159.385 152.4 90)
+			(effects
+				(font
+					(size 1.27 1.27)
+				)
+				(hide yes)
+			)
+		)
+		(property "Datasheet" "~"
+			(at 159.385 152.4 90)
 			(effects
 				(font
@@
 		)
 		(property "Description" "RJ connector, 6P6C (6 positions 6 connected), RJ12/RJ18/RJ25"
-			(at 161.29 152.4 0)
+			(at 158.75 152.4 0)
 			(effects
 				(font
@@
 	(symbol
 		(lib_id "Connector:6P6C")
-		(at 226.06 152.4 90)
-		(unit 1)
-		(exclude_from_sim no)
-		(in_bom yes)
-		(on_board yes)
-		(dnp no)
-		(fields_autoplaced yes)
+		(at 223.52 152.4 270)
+		(mirror x)
+		(unit 1)
+		(exclude_from_sim no)
+		(in_bom yes)
+		(on_board yes)
+		(dnp no)
 		(property "Reference" "J20"
-			(at 234.95 151.1299 90)
+			(at 214.63 151.1299 90)
 			(effects
 				(font
@@
 		)
 		(property "Value" "6P6C"
-			(at 234.95 153.6699 90)
-			(effects
-				(font
-					(size 1.27 1.27)
-				)
-				(justify right)
-			)
-		)
-		(property "Footprint" ""
-			(at 225.425 152.4 90)
-			(effects
-				(font
-					(size 1.27 1.27)
-				)
-				(hide yes)
-			)
-		)
-		(property "Datasheet" "~"
-			(at 225.425 152.4 90)
+			(at 214.63 153.6699 90)
+			(effects
+				(font
+					(size 1.27 1.27)
+				)
+				(justify right)
+			)
+		)
+		(property "Footprint" ""
+			(at 224.155 152.4 90)
+			(effects
+				(font
+					(size 1.27 1.27)
+				)
+				(hide yes)
+			)
+		)
+		(property "Datasheet" "~"
+			(at 224.155 152.4 90)
 			(effects
 				(font
@@
 		)
 		(property "Description" "RJ connector, 6P6C (6 positions 6 connected), RJ12/RJ18/RJ25"
-			(at 226.06 152.4 0)
-			(effects
-				(font
+			(at 223.52 152.4 0)
+			(effects
+				(font
